Commit message: start of ikin stuff

File: hw5code/urdf/robot_approx.urdf (robot description, URDF)
Before this commit: robot robot, 15 links, 14 joints
Joints:
- joint connect-motor0output-motor1base: origin xyz=0 0 0.081 rpy=0 1.57 0 -> xyz=0 0 0.1 rpy=0 1.57 0
- joint connect-motor2output-motor3base: origin xyz=0 -0.3 0 rpy=0 0 0 -> xyz=0 0.3 0 rpy=0 0 0
