Commit message: after friday demos

File: tunecode/urdf/robot.urdf (robot description, URDF)
Before this commit: robot robot, 15 links, 14 joints
Links:
- removed link motor3base
- removed link motor3output
- removed link motor4base
- removed link motor4output
- added link link1part1; visual box size=0.05 0.08 0.005
- added link link1part2; visual box size=0.05 0.005 0.075
- added link link2; visual box size=0.55 0.05 0.005
- added link link3; visual box size=0.5 0.05 0.005
- added link motor0; visual mesh filename=package://hebiros_description/meshes/x5.stl scale=0.001 0.001 0.001
- added link motor1; visual mesh filename=package://hebiros_description/meshes/x5.stl scale=0.001 0.001 0.001
- added link motor2; visual mesh filename=package://hebiros_description/meshes/x5.stl scale=0.001 0.001 0.001
- added link table; visual box size=0.5 0.5 0.05
Joints:
- removed joint Boogaloo/elbow
- removed joint Boogaloo/shoulder
- removed joint Boogaloo/twist
- removed joint Boogaloo/wrist
- removed joint Boogaloo/yaw
- removed joint connect-motor2output-motor3base
- removed joint connect-motor3output-motor4base
- removed joint connect-motor4output-tip
- added joint Dwarfs/Doc: type continuous, parent motor0base, child motor0output, axis 0 0 1
- added joint Dwarfs/Grumpy: type continuous, parent motor2base, child motor2output, axis 0 0 1
- added joint Dwarfs/Sleepy: type continuous, parent motor1base, child motor1output, axis 0 0 -1
- added joint attach-motor0: type fixed, parent motor0base, child motor0
- added joint attach-motor1: type fixed, parent motor1base, child motor1
- added joint attach-motor2: type fixed, parent motor2base, child motor2
- added joint connect-motor0output-link1part1: type fixed, parent motor0output, child link1part1
- added joint connect-motor0output-link1part2: type fixed, parent motor0output, child link1part2
- added joint connect-motor1output-link2: type fixed, parent motor1output, child link2
- added joint connect-motor2output-link3: type fixed, parent motor2output, child link3
- added joint connect-motor2output-tip: type fixed, parent motor2output, child tip, origin xyz=0.5 0 0.0335 rpy=0 1.57 0
- added joint connect-world-table: type fixed, parent world, child table
- joint connect-motor0output-motor1base: origin xyz=0 -0.051 0.051 rpy=1.57 1.57 0 -> xyz=0 0.05 0.081 rpy=1.57 0 0
- joint connect-motor1output-motor2base: origin xyz=-0.606 0 -0.064 rpy=0 0 0 -> xyz=0.5 0 0.036 rpy=0 0 0
- joint connect-world-motor0base: origin xyz=0 -0.124 0.081 rpy=0 0 0 -> xyz=0 0 0 rpy=0 0 0
