Commit message: redid ikin with trig

File: boogaloo/urdf/robot_approx.urdf (robot description, URDF)
Before this commit: robot robot, 15 links, 14 joints
Joints:
- joint connect-motor0output-motor1base: origin xyz=0 0 0.081 rpy=0 1.57 0 -> xyz=0 0 0.1 rpy=1.57 1.57 0
- joint connect-motor2output-motor3base: origin xyz=0 -0.3 0 rpy=0 0 0 -> xyz=0 0.3 0 rpy=3.14 0 0
- joint connect-motor4output-tip: origin xyz=0 0 0.1 rpy=0 0 0 -> xyz=0 0 0.1 rpy=0 0 3.14
- joint connect-world-motor0base: origin xyz=0 0.1 0 rpy=0 0 0 -> xyz=0 -0.1 .1 rpy=0 0 0

Commit message: first pass on throwing

File: boogaloo/urdf/robot_approx.urdf (robot description, URDF)
Before this commit: robot robot, 15 links, 14 joints
Joints:
- joint connect-motor0output-motor1base: origin xyz=0 -0.051 0.051 rpy=1.57 1.57 0 -> xyz=0 -0.049 0.062 rpy=1.57 1.57 0
- joint connect-motor1output-motor2base: origin xyz=-0.606 0 -0.064 rpy=0 0 0 -> xyz=-0.600 0 -0.062 rpy=0 0 0
- joint connect-motor2output-motor3base: origin xyz=0 0.298 0 rpy=3.14 0 0 -> xyz=0 0.294 0 rpy=3.14 0 0
- joint connect-motor3output-motor4base: origin xyz=0.038 0 0.110 rpy=0 1.57 0 -> xyz=0.040 0 0.108 rpy=0 1.57 0
- joint connect-motor4output-tip: origin xyz=0 0 0.056 rpy=0 0 3.14 -> xyz=0 0 0.080 rpy=0 0 3.14
- joint connect-world-motor0base: origin xyz=0 -0.124 0.081 rpy=0 0 0 -> xyz=0 -0.122 0.081 rpy=0 0 0
